Commit message: 6.4 upd

File: lab6/ex04/robot_description/urdf/robot.urdf.xacro (robot description, xacro)
@@ -22,15 +22,9 @@
         <color rgba="1 1 1 1" />
     </material>
-    <material name="orange">
-        <color rgba="1 0.1 1 1"/>
-    </material>
-    <material name="blue">
-        <color rgba="0.2 0.2 1 1"/>
-    </material>
     <material name="black">
         <color rgba="0 0 0 1"/>
     </material>
-    <material name="red">
-        <color rgba="1 0 0 1"/>
+    <material name="green">
+        <color rgba="0 1 0 1"/>
     </material>
     <link name="base_link">
@@ -61,5 +55,5 @@
             <box size="${chassis_length} ${chassis_width} ${chassis_height}"/>
         </geometry>
-        <material name="orange"/>
+        <material name="green"/>
     </visual>
     <collision>
@@ -71,5 +65,5 @@
     </link>
     <gazebo reference="chassis">
-        <material>Gazebo/Orange</material>
+        <material>Gazebo/Green</material>
     </gazebo>
     <joint name="left_wheel_joint" type="continuous">
@@ -84,5 +78,5 @@
                 <cylinder radius="${wheel_radius}" length="${wheel_thickness}"/>
             </geometry>
-            <material name="blue"/>
+            <material name="black"/>
         </visual>
         <collision>
@@ -100,5 +94,5 @@
     </link>
     <gazebo reference="left_wheel">
-        <material>Gazebo/Blue</material>
+        <material>Gazebo/Black</material>
     </gazebo>
     <joint name="right_wheel_joint" type="continuous">
@@ -113,5 +107,5 @@
                 <cylinder radius="${wheel_radius}" length="${wheel_thickness}"/>
             </geometry>
-            <material name="blue"/>
+            <material name="black"/>
         </visual>
         <collision>
@@ -129,5 +123,5 @@
     </link>
     <gazebo reference="right_wheel">
-        <material>Gazebo/Blue</material>
+        <material>Gazebo/Black</material>
     </gazebo>
     <joint name="caster_wheel_joint" type="fixed">
